Commit message: Initial import of gazebo setup, loads, but physics incorrect and needs testing

File: widowx_arm_description/robots/widowx_arm.urdf.xacro (robot description, xacro)
@@ -1,4 +1,5 @@
 <?xml version="1.0" ?>
 <robot name="widowx_arm" xmlns:xacro="http://ros.org/wiki/xacro">
+        <xacro:include filename="$(find widowx_arm_description)/urdf/gazebo.urdf.xacro"/>
 	<xacro:include filename="$(find widowx_arm_description)/urdf/widowx.urdf.xacro"/>
 	<link name="base_footprint">

File: widowx_arm_description/urdf/widowx.urdf.xacro (robot description, xacro)
@@ -277,5 +277,7 @@
   <transmission name="tran1">
     <type>transmission_interface/SimpleTransmission</type>
-    <joint name="joint_1"/>
+    <joint name="joint_1">
+	<hardwareInterface>hardware_interface/PositionJointInterface</hardwareInterface>
+    </joint>
     <actuator name="motor1">
       <hardwareInterface>EffortJointInterface</hardwareInterface>
@@ -285,5 +287,7 @@
  <transmission name="tran2">
     <type>transmission_interface/SimpleTransmission</type>
-    <joint name="joint_2"/>
+    <joint name="joint_2">
+	<hardwareInterface>hardware_interface/PositionJointInterface</hardwareInterface>
+    </joint>
     <actuator name="motor2">
       <hardwareInterface>EffortJointInterface</hardwareInterface>
@@ -293,5 +297,7 @@
  <transmission name="tran3">
     <type>transmission_interface/SimpleTransmission</type>
-    <joint name="joint_3"/>
+    <joint name="joint_3">
+	<hardwareInterface>hardware_interface/PositionJointInterface</hardwareInterface>
+    </joint>
     <actuator name="motor3">
       <hardwareInterface>EffortJointInterface</hardwareInterface>
@@ -301,5 +307,7 @@
  <transmission name="tran4">
     <type>transmission_interface/SimpleTransmission</type>
-    <joint name="joint_4"/>
+    <joint name="joint_4">
+	<hardwareInterface>hardware_interface/PositionJointInterface</hardwareInterface>
+    </joint>
     <actuator name="motor4">
       <hardwareInterface>EffortJointInterface</hardwareInterface>
@@ -309,5 +317,7 @@
  <transmission name="tran5">
     <type>transmission_interface/SimpleTransmission</type>
-    <joint name="joint_6"/>
+    <joint name="joint_5">
+	<hardwareInterface>hardware_interface/PositionJointInterface</hardwareInterface>
+    </joint>
     <actuator name="motor5">
       <hardwareInterface>EffortJointInterface</hardwareInterface>
@@ -317,5 +327,7 @@
  <transmission name="tran6">
     <type>transmission_interface/SimpleTransmission</type>
-    <joint name="gripper_prismatic_joint_1"/>
+    <joint name="gripper_prismatic_joint_2">
+	<hardwareInterface>hardware_interface/PositionJointInterface</hardwareInterface>
+    </joint>
     <actuator name="motor6">
       <hardwareInterface>EffortJointInterface</hardwareInterface>
