Commit message: RViz is now able to control the arm simulated in gazebo
Added a new launch file for this specific gazebo + rviz use case

File: widowx_arm_description/urdf/widowx.urdf.xacro (robot description, xacro)
@@ -327,5 +327,5 @@
  <transmission name="tran6">
     <type>transmission_interface/SimpleTransmission</type>
-    <joint name="gripper_prismatic_joint_2">
+    <joint name="gripper_joint">
 	<hardwareInterface>hardware_interface/PositionJointInterface</hardwareInterface>
     </joint>

Commit message: Update limits to match the physical widowx

File: widowx_arm_description/urdf/widowx.urdf.xacro (robot description, xacro)
@@ -212,5 +212,5 @@
          <child link="${prefix}biceps_link" />
          <axis xyz="0 1 0" />
-         <limit lower="-1.571" upper="1.571" effort="6" velocity="1.571" />
+         <limit lower="-1.689" upper="1.689" effort="6" velocity="1.571" />
       </joint>
       <joint name="${prefix}joint_3" type="revolute">
@@ -219,5 +219,5 @@
          <child link="${prefix}forearm_link" />
          <axis xyz="0 1 0" />
-         <limit lower="-1.571" upper="1.571" effort="6" velocity="1.571" />
+         <limit lower="-2.83" upper="1.658" effort="6" velocity="1.571" />
       </joint>
       <joint name="${prefix}joint_4" type="revolute">
@@ -226,5 +226,5 @@
          <child link="${prefix}wrist_1_link" />
          <axis xyz="0 1 0" />
-         <limit lower="-1.745" upper="1.745" effort="6" velocity="1.571" />
+         <limit lower="-1.875" upper="1.973" effort="6" velocity="1.571" />
       </joint>
       <joint name="${prefix}joint_5" type="revolute">

Commit message: Guestimate inertial parameters for the arm
These values produce believable movement in gazebo.

File: widowx_arm_description/urdf/widowx.urdf.xacro (robot description, xacro)
@@ -27,6 +27,6 @@
          <inertial>
             <origin xyz="0 0 0" rpy="0 0 0" />
-            <mass value="1" />
-            <inertia ixx="1.0" ixy="0.0" ixz="0.0" iyy="1.0" iyz="0.0" izz="1.0" />
+            <mass value="0.75" />
+            <inertia ixx="0.00219844" ixy="0.0" ixz="0.0" iyy="0.00219844" iyz="0.0" izz="0.00338438" />
          </inertial>
       </link>
@@ -47,6 +47,6 @@
          <inertial>
             <origin xyz="0 0 0" rpy="0 0 0" />
-            <mass value="1" />
-            <inertia ixx="1.0" ixy="0.0" ixz="0.0" iyy="1.0" iyz="0.0" izz="1.0" />
+            <mass value="0.08" />
+            <inertia ixx="0.00007227" ixy="0.0" ixz="0.0" iyy="0.00007227" iyz="0.0" izz="0.00012321" />
          </inertial>
       </link>
@@ -67,6 +67,6 @@
          <inertial>
             <origin xyz="0 0 0" rpy="0 0 0" />
-            <mass value="1" />
-            <inertia ixx="1.0" ixy="0.0" ixz="0.0" iyy="1.0" iyz="0.0" izz="1.0" />
+            <mass value="0.270" />
+            <inertia ixx="0.00091125" ixy="0.0" ixz="0.0" iyy="0.00078525" iyz="0.0" izz="0.00023850" />
          </inertial>
       </link>
@@ -87,6 +87,6 @@
          <inertial>
             <origin xyz="0 0 0" rpy="0 0 0" />
-            <mass value="1" />
-            <inertia ixx="1.0" ixy="0.0" ixz="0.0" iyy="1.0" iyz="0.0" izz="1.0"/>
+            <mass value="0.130" />
+            <inertia ixx="0.00030442" ixy="0.0" ixz="0.0" iyy="0.00029467" iyz="0.0" izz="0.00004442"/>
          </inertial>
       </link>
@@ -107,6 +107,6 @@
          <inertial>
             <origin xyz="0 0 0" rpy="0 0 0" />
-            <mass value="1" />
-            <inertia ixx="1.0" ixy="0.0" ixz="0.0" iyy="1.0" iyz="0.0" izz="1.0" />
+            <mass value="0.085" />
+            <inertia ixx="0.00006304" ixy="0.0" ixz="0.0" iyy="0.00005667" iyz="0.0" izz="0.00002904" />
          </inertial>
       </link>
@@ -127,6 +127,6 @@
          <inertial>
             <origin xyz="0 0 0" rpy="0 0 0" />
-            <mass value="1" />
-            <inertia ixx="1.0" ixy="0.0" ixz="0.0" iyy="1.0" iyz="0.0" izz="1.0" />
+            <mass value="0.065" />
+            <inertia ixx="0.00002708" ixy="0.0" ixz="0.0" iyy="0.00001842" iyz="0.0" izz="0.00001842" />
          </inertial>
       </link>

File: widowx_arm_description/urdf/widowx_gripper.xacro (robot description, xacro)
@@ -17,6 +17,6 @@
       <inertial>
          <origin xyz="0 0 0" rpy="0 0 0" />
-         <mass value="1" />
-         <inertia ixx="1.0" ixy="0.0" ixz="0.0" iyy="1.0" iyz="0.0" izz="1.0" />
+         <mass value="0.01" />
+         <inertia ixx="0.00000417" ixy="0.0" ixz="0.0" iyy="0.00000142" iyz="0.0" izz="0.00000542" />
       </inertial>
    </link>
@@ -39,6 +39,6 @@
       <inertial>
          <origin xyz="0 0 0" rpy="0 0 0" />
-         <mass value="1" />
-         <inertia ixx="1.0" ixy="0.0" ixz="0.0" iyy="1.0" iyz="0.0" izz="1.0" />
+         <mass value="0.005" />
+         <inertia ixx="0.00000083" ixy="0.0" ixz="0.0" iyy="0.00000133" iyz="0.0" izz="0.00000083" />
       </inertial>
    </link>
@@ -59,6 +59,6 @@
       <inertial>
          <origin xyz="0 0 0" rpy="0 0 0" />
-         <mass value="1" />
-         <inertia ixx="1.0" ixy="0.0" ixz="0.0" iyy="1.0" iyz="0.0" izz="1.0" />
+         <mass value="0.005" />
+         <inertia ixx="0.00000083" ixy="0.0" ixz="0.0" iyy="0.00000133" iyz="0.0" izz="0.00000083" />
       </inertial>
    </link>
