Commit message: Require the use of the mimic joint plugin
from: https://github.com/roboticsgroup/roboticsgroup_gazebo_plugins

This is needed for the gripper's fingers to match their motion

File: widowx_arm_description/urdf/gazebo.urdf.xacro (robot description, xacro)
@@ -3,4 +3,8 @@
   <gazebo>
     <plugin name="ros_control" filename="libgazebo_ros_control.so"/>
+    <plugin name="mimic_joint" filename="libroboticsgroup_gazebo_mimic_joint_plugin.so">
+	<joint>gripper_joint</joint>
+	<mimicJoint>gripper_prismatic_joint_2</mimicJoint>
+    </plugin>
   </gazebo>
   <xacro:macro name="ur_arm_gazebo" params="prefix"/>

Commit message: Don't need this tag

File: widowx_arm_description/urdf/gazebo.urdf.xacro (robot description, xacro)
@@ -8,4 +8,3 @@
     </plugin>
   </gazebo>
-  <xacro:macro name="ur_arm_gazebo" params="prefix"/>
 </robot>
