Commit message: Halve the gripper's width so that both simulation and reality match
This requires halving the goal width you send to the gripper's goal node

(ie. if you want a width X, send X / 2 )

File: widowx_arm_description/urdf/widowx_gripper.xacro (robot description, xacro)
@@ -74,5 +74,5 @@
       <child link="${prefix}gripper_1_link" />
       <axis xyz="0 -1 0" />
-      <limit lower="0.002" upper="0.031" effort="0" velocity="0.5" />
+      <limit lower="0.001" upper="0.0158" effort="0" velocity="0.5" />
    </joint>
    <joint name="${prefix}gripper_prismatic_joint_2" type="prismatic">
@@ -82,5 +82,5 @@
       <mimic joint="${prefix}gripper_joint" />
       <axis xyz="0 1 0" />
-      <limit lower="0.002" upper="0.031" effort="0" velocity="0.5" />
+      <limit lower="0.001" upper="0.0158" effort="0" velocity="0.5" />
    </joint>
 </robot>

Commit message: Add friction onto the gripper's fingers

File: widowx_arm_description/urdf/widowx_gripper.xacro (robot description, xacro)
@@ -84,3 +84,45 @@
       <limit lower="0.001" upper="0.0158" effort="0" velocity="0.5" />
    </joint>
+      <gazebo reference="${prefix}gripper_1_link">
+        <collision><surface>
+                <bounce><threshold>100000</threshold></bounce>
+        <friction>
+        <ode>
+                <mu>10000000</mu>
+                <mu2>10000000</mu2>
+                <slip1>0.0</slip1>
+                <slip2>0.0</slip2>
+        </ode>
+        <bullet>
+                <friction>10000000</friction>
+                <friction2>10000000</friction2>
+        </bullet>
+        </friction>
+        <contact>
+                <ode><kd>100</kd></ode>
+                <bullet><kp>1000000000</kp><kd>100</kd><soft_erp>0.20</soft_erp></bullet>
+        </contact>
+        </surface></collision>
+      </gazebo>
+      <gazebo reference="${prefix}gripper_2_link">
+        <collision><surface>
+                <bounce><threshold>100000</threshold></bounce>
+        <friction>
+        <ode>
+                <mu>10000000</mu>
+                <mu2>10000000</mu2>
+                <slip1>0.0</slip1>
+                <slip2>0.0</slip2>
+        </ode>
+        <bullet>
+                <friction>10000000</friction>
+                <friction2>10000000</friction2>
+        </bullet>
+        </friction>
+        <contact>
+                <ode><kd>100</kd></ode>
+                <bullet><kp>1000000000</kp><kd>100</kd><soft_erp>0.20</soft_erp></bullet>
+        </contact>
+        </surface></collision>
+      </gazebo>
 </robot>
